File: smart road pcb/smart road pcb.kicad_pcb (KiCad board)
At the start: 2 copper layers, 107.5 x 58.5 mm, 9 parts, among them U1 ESP32-DEVKITC-32D, U2 ESP32-CAM

Commit message: edit PCB and making case
Parts:
- added BT1: BC3AAAPC, BC3AAAPC:BAT_BC3AAAPC, F.Cu at (203.4, 127.2)
- added C1: C, Capacitor_THT:C_Disc_D5.0mm_W2.5mm_P5.00mm, F.Cu at (157.0, 132.0)
- added C2: C, Capacitor_THT:CP_Radial_D5.0mm_P2.50mm, F.Cu at (152.0, 113.5)
- added U4: LD1117V33, Package_TO_SOT_THT:TO-220-3_Vertical, F.Cu at (151.9, 123.0)
Connections:
- U1 pad J2-1: unconnected-(U1-3V3-PadJ2-1) -> B3V3
- U1 pad J3-1: unconnected-(U1-GND3-PadJ3-1) -> -
- U1 pad J3-11: unconnected-(U1-IO17-PadJ3-11) -> ESP_TX_RX
- U1 pad J3-12: unconnected-(U1-IO16-PadJ3-12) -> ESP_RX_TX
- U2 pad P$1: unconnected-(U2-GND@1-PadP$1) -> -
- U2 pad P$11: unconnected-(U2-GPIO12-PadP$11) -> ESP_RX_TX
- U2 pad P$12: unconnected-(U2-GPIO13-PadP$12) -> ESP_TX_RX
- U2 pad P$8: unconnected-(U2-3V3-PadP$8) -> B3V3
Routing:
- net -: track 0.00 -> 149.7 mm, vias 0 -> 1
- net B3V3: track 0.00 -> 119.8 mm
- net +: track 0.00 -> 81.6 mm
- net ESP_TX_RX: track 0.00 -> 68.5 mm
- net ESP_RX_TX: track 0.00 -> 66.1 mm
Other:
- board size 107.5 x 58.5 mm -> 107.5 x 105.5 mm
