File: smart road pcb/smart road pcb.kicad_sch (KiCad schematic)
At the start: 8 parts, among them U1 ESP32-DEVKITC-32D, U2 ESP32-CAM

Commit message: edit PCB and making case
Parts:
- added BT1: BC3AAAPC, BC3AAAPC:BAT_BC3AAAPC, symbol BC3AAAPC:BC3AAAPC
- added C1: C, Capacitor_THT:C_Disc_D5.0mm_W2.5mm_P5.00mm, symbol Device:C
- added C2: C, Capacitor_THT:CP_Radial_D5.0mm_P2.50mm, symbol Device:C
- added U4: LD1117V33, Package_TO_SOT_THT:TO-220-3_Vertical, symbol Regulator_Linear:LD1117V33
Connections:
- net B3V3: now reaches U1.J2-1 (3V3)
- net B3V3: now also U2.P$8 (3V3), C2.2, U4.2 (VO)
- net -: now reaches U1.J3-1 (GND3)
- net -: now also U2.P$1 (GND@1), BT1.-, C1.2, C2.1, U4.1 (GND)
- net ESP_TX_RX: now reaches U1.J3-11 (IO17)
- net ESP_TX_RX: now also U2.P$12 (GPIO13)
- net ESP_RX_TX: now reaches U1.J3-12 (IO16)
- net ESP_RX_TX: now also U2.P$11 (GPIO12)
- new net +: BT1.+, C1.1, U4.3 (VI)
